Commit message: 添加了amcl定位模块

File: src/gazebo_sim/xacro/base.xacro (robot description, xacro)
@@ -44,5 +44,5 @@
     <xacro:property name="wheel_radius" value="0.0325" />
     <xacro:property name="wheel_length" value="0.015" />
-    <xacro:property name="wheel_m" value="0.05" />
+    <xacro:property name="wheel_m" value="0.5" />
     <xacro:macro name="add_wheels" params="name flag">
       <link name="${name}_wheel">
